Commit message: 🎖️ Updates kinematics and models

File: simulation/model.urdf (robot description, URDF)
Before this commit: robot robot, 19 links, 18 joints
Links:
- link back_left_foot_link: geometry collision sphere radius=0.1; visual mesh filename=package://stl/foot.stl scale=0.01 0.01 0.01
- link back_left_shoulder_link: geometry collision box size=0.044 0.038 0.25; visual mesh filename=package://stl/joint.stl scale=0.01 0.01 0.01
- link back_right_foot_link: geometry collision sphere radius=0.1; visual mesh filename=package://stl/foot.stl scale=0.01 0.01 0.01
- link back_right_shoulder_link: geometry collision box size=0.044 0.038 0.25; visual mesh filename=package://stl/joint.stl scale=0.01 0.01 0.01
- link base_link: geometry collision box size=0.6 1.4 0.25; visual mesh filename=package://stl/body.stl scale=0.01 0.01 0.01
- link front_left_foot_link: geometry collision sphere radius=0.1; visual mesh filename=package://stl/foot.stl scale=0.01 0.01 0.01
- link front_left_shoulder_link: geometry collision box size=0.044 0.038 0.25; visual mesh filename=package://stl/joint.stl scale=0.01 0.01 0.01
- link front_right_foot_link: geometry collision sphere radius=0.1; visual mesh filename=package://stl/foot.stl scale=0.01 0.01 0.01
- link front_right_shoulder_link: geometry collision box size=0.044 0.038 0.25; visual mesh filename=package://stl/joint.stl scale=0.01 0.01 0.01
- link middle_left_foot_link: geometry collision sphere radius=0.1; visual mesh filename=package://stl/foot.stl scale=0.01 0.01 0.01
- link middle_left_shoulder_link: geometry collision box size=0.044 0.038 0.25; visual mesh filename=package://stl/joint.stl scale=0.01 0.01 0.01
- link middle_right_foot_link: geometry collision sphere radius=0.1; visual mesh filename=package://stl/foot.stl scale=0.01 0.01 0.01
- link middle_right_shoulder_link: geometry collision box size=0.044 0.038 0.25; visual mesh filename=package://stl/joint.stl scale=0.01 0.01 0.01

File: simulation/model.xacro (robot description, xacro)
@@ -11,7 +11,7 @@
     </material>
     <!-- Params -->
-    <xacro:property name="body_length" value="0.140" />
-    <xacro:property name="body_width" value="0.110" />
-    <xacro:property name="body_height" value="0.070" />
+    <xacro:property name="body_length" value="1.4" />
+    <xacro:property name="body_width" value="0.6" />
+    <xacro:property name="body_height" value="0.25" />
     <xacro:property name="shoulder_length" value="0.044" />
     <xacro:property name="shoulder_width" value="0.038" />
@@ -48,5 +48,5 @@
                     <box size="${shoulder_length} ${shoulder_width} ${body_height}" />
                 </geometry>
-                <origin rpy="0 0 0" xyz="0 0 0" />
+                <origin rpy="0 0 0" xyz="0 0 0.6" />
             </collision>
             <inertial>
@@ -78,7 +78,7 @@
             <collision>
                 <geometry>
-                    <box size="0.026 0.020 ${foot_length}" />
+                    <sphere radius="0.1" />
                 </geometry>
-                <origin rpy="0.0 0.0 0.0" xyz="0.0 0.0 -0.050" />
+                <origin rpy="0 0 0" xyz="-0.5 0.98 0.0225" />
             </collision>
             <inertial>
@@ -140,7 +140,7 @@
         <collision>
             <geometry>
-                <box size="${body_length} ${body_width} ${body_height}" />
+                <box size="${body_width} ${body_length} ${body_height}" />
             </geometry>
-            <origin rpy="0 0 0" xyz="0 0 0" />
+            <origin rpy="0 0 0" xyz="0 0 0.6" />
         </collision>
         <inertial>
