Commit message: 🦋 Updates masses and motor forces for simulation

File: simulation/model.xacro (robot description, xacro)
@@ -18,5 +18,5 @@
     <xacro:property name="leg_length" value="0.1075" />
     <xacro:property name="foot_length" value="0.130" />
-    <xacro:property name="toe_radius" value="0.020" />
+    <xacro:property name="toe_radius" value="0.1" />
     <xacro:property name="toe_width" value="0.020" />
     <xacro:property name="shift" value="-1.015" />
@@ -51,6 +51,6 @@
             </collision>
             <inertial>
-                <mass value="0.10" />
-                <inertia ixx="100" ixy="0" ixz="0" iyy="100" iyz="0" izz="100" />
+                <mass value="0.01" />
+                <inertia ixx="0.0001" ixy="0" ixz="0" iyy="0.0001" iyz="0" izz="0.0001" />
             </inertial>
         </link>
@@ -78,11 +78,12 @@
             <collision>
                 <geometry>
-                    <sphere radius="0.1" />
+                    <sphere radius="${toe_radius}" />
                 </geometry>
-                <origin rpy="0 0 0" xyz="-0.5 0.98 0.0225" />
+                <origin rpy="0 0 0" xyz="-0.8 0.98 0.0225" />
+                <contact_coefficients mu="1.1" />
             </collision>
             <inertial>
-                <mass value="0.1" />
-                <inertia ixx="1000" ixy="0" ixz="0" iyy="1000" iyz="0" izz="1000" />
+                <mass value="0.01" />
+                <inertia ixx="0.0001" ixy="0" ixz="0" iyy="0.0001" iyz="0" izz="0.0001" />
             </inertial>
         </link>
@@ -105,5 +106,5 @@
             <axis xyz="0 1 0" />
             <origin rpy="0 0 0" xyz="-0.28 ${shift} 0.59" />
-            <limit effort="1000.0" lower="-2.666" upper="1.548" velocity="0.5" />
+            <limit effort="1000.0" lower="-2.666" upper="1.548" velocity="1" />
             <dynamics damping="0.0" friction="0.0" />
         </joint>
@@ -115,5 +116,5 @@
             <axis xyz="0 1 0" />
             <origin rpy="0 0 0" xyz="-0.43 0 -0" />
-            <limit effort="1000.0" lower="-2.6" upper="0.1" velocity="0.5" />
+            <limit effort="1000.0" lower="-2.6" upper="0.1" velocity="1" />
             <dynamics damping="0.0" friction="0.5" />
         </joint>
@@ -145,6 +146,6 @@
         </collision>
         <inertial>
-            <mass value="2.80" />
-            <inertia ixx="100" ixy="0" ixz="0" iyy="100" iyz="0" izz="100" />
+            <mass value="0.05" />
+            <inertia ixx="0.0001" ixy="0" ixz="0" iyy="0.0001" iyz="0" izz="0.0001" />
         </inertial>
     </link>
