Commit message: 🐉 Adds inertia to model

File: simulation/src/resources/model.urdf (robot description, URDF)
Before this commit: robot robot, 19 links, 18 joints
Links:
- link back_left_foot_link: mass 0.1 -> 0.01
- link back_left_leg_link: mass None -> 0.01; geometry collision box size=0.1075 0.1075 0.1075; visual mesh filename=package://stl/middle_joint.stl scale=0.01 0.01 0.01
- link back_left_shoulder_link: mass 0.10 -> 0.01
- link back_right_foot_link: mass 0.1 -> 0.01
- link back_right_leg_link: mass None -> 0.01; geometry collision box size=0.1075 0.1075 0.1075; visual mesh filename=package://stl/middle_joint.stl scale=0.01 0.01 0.01
- link back_right_shoulder_link: mass 0.10 -> 0.01
- link base_link: mass 2.80 -> 0.05
- link front_left_foot_link: mass 0.1 -> 0.01
- link front_left_leg_link: mass None -> 0.01; geometry collision box size=0.1075 0.1075 0.1075; visual mesh filename=package://stl/middle_joint.stl scale=0.01 0.01 0.01
- link front_left_shoulder_link: mass 0.10 -> 0.01
- link front_right_foot_link: mass 0.1 -> 0.01
- link front_right_leg_link: mass None -> 0.01; geometry collision box size=0.1075 0.1075 0.1075; visual mesh filename=package://stl/middle_joint.stl scale=0.01 0.01 0.01
- link front_right_shoulder_link: mass 0.10 -> 0.01
- link middle_left_foot_link: mass 0.1 -> 0.01
- link middle_left_leg_link: mass None -> 0.01; geometry collision box size=0.1075 0.1075 0.1075; visual mesh filename=package://stl/middle_joint.stl scale=0.01 0.01 0.01
- link middle_left_shoulder_link: mass 0.10 -> 0.01
- link middle_right_foot_link: mass 0.1 -> 0.01
- link middle_right_leg_link: mass None -> 0.01; geometry collision box size=0.1075 0.1075 0.1075; visual mesh filename=package://stl/middle_joint.stl scale=0.01 0.01 0.01
- link middle_right_shoulder_link: mass 0.10 -> 0.01
Joints:
- joint back_left_foot: limit lower=-2.6 upper=0.1 effort=1000.0 velocity=0.5 -> lower=-2.6 upper=0.1 effort=1000.0 velocity=1
- joint back_left_leg: limit lower=-2.666 upper=1.548 effort=1000.0 velocity=0.5 -> lower=-2.666 upper=1.548 effort=1000.0 velocity=1
- joint back_right_foot: limit lower=-2.6 upper=0.1 effort=1000.0 velocity=0.5 -> lower=-2.6 upper=0.1 effort=1000.0 velocity=1
- joint back_right_leg: limit lower=-2.666 upper=1.548 effort=1000.0 velocity=0.5 -> lower=-2.666 upper=1.548 effort=1000.0 velocity=1
- joint front_left_foot: limit lower=-2.6 upper=0.1 effort=1000.0 velocity=0.5 -> lower=-2.6 upper=0.1 effort=1000.0 velocity=1
- joint front_left_leg: limit lower=-2.666 upper=1.548 effort=1000.0 velocity=0.5 -> lower=-2.666 upper=1.548 effort=1000.0 velocity=1
- joint front_right_foot: limit lower=-2.6 upper=0.1 effort=1000.0 velocity=0.5 -> lower=-2.6 upper=0.1 effort=1000.0 velocity=1
- joint front_right_leg: limit lower=-2.666 upper=1.548 effort=1000.0 velocity=0.5 -> lower=-2.666 upper=1.548 effort=1000.0 velocity=1
- joint middle_left_foot: limit lower=-2.6 upper=0.1 effort=1000.0 velocity=0.5 -> lower=-2.6 upper=0.1 effort=1000.0 velocity=1
- joint middle_left_leg: limit lower=-2.666 upper=1.548 effort=1000.0 velocity=0.5 -> lower=-2.666 upper=1.548 effort=1000.0 velocity=1
- joint middle_right_foot: limit lower=-2.6 upper=0.1 effort=1000.0 velocity=0.5 -> lower=-2.6 upper=0.1 effort=1000.0 velocity=1
- joint middle_right_leg: limit lower=-2.666 upper=1.548 effort=1000.0 velocity=0.5 -> lower=-2.666 upper=1.548 effort=1000.0 velocity=1

File: simulation/src/resources/model.xacro (robot description, xacro)
@@ -17,4 +17,6 @@
     <xacro:property name="shoulder_width" value="0.038" />
     <xacro:property name="leg_length" value="0.1075" />
+    <xacro:property name="leg_width" value="0.1075" />
+    <xacro:property name="leg_height" value="0.1075" />
     <xacro:property name="foot_length" value="0.130" />
     <xacro:property name="toe_radius" value="0.1" />
@@ -65,4 +67,14 @@
                 <material name="body_color" />
             </visual>
+            <collision>
+                <geometry>
+                    <box size="${leg_length} ${leg_width} ${leg_height}" />
+                </geometry>
+                <origin rpy="0 0 0" xyz="0 0 0.6" />
+            </collision>
+            <inertial>
+                <mass value="0.01" />
+                <inertia ixx="0.0001" ixy="0" ixz="0" iyy="0.0001" iyz="0" izz="0.0001" />
+            </inertial>
         </link>
     </xacro:macro>
